File: PCB/Vac_Pump_Controller/Vac_Pump_Controller.kicad_sch (KiCad schematic)
At the start: 21 parts, among them J1 Conn_01x04_Socket, J1A Conn_01x04_Pin, J2 Conn_01x02_Socket, J2A Conn_01x02_Pin, J3 Conn_01x08_Socket, J3A Conn_01x08_Pin, J4 AC Plug, J5 DIN-6, J6 Conn_01x06_Socket, J6A Conn_01x06_Pin, J7 DIN-6, K1 Dual Relay Module, SW1 RotaryEncoder_Switch_MP, SW2 Pwr Switch, U1 WeMos D1 Mini32, U2 JXI 1.28in Round LCD

Commit message: Baseline: as-validated bench config
Alarm IO22->IO33 (matches validated hw); MPXV6115VC6U documented; title block + attribution; ERC clean (PWR_FLAGs, AC plug pins numbered); KiCad 10 format
Parts:
- renumbered J1A to J1A1, J2A to J2A1, J3A to J3A1, J6A to J6A1
Connections:
- net Alarm: now also U1.30 (IO33); no longer U1.6 (IO22)
- net Earth: now also J4.3 (PE); no longer J4. (PE)
- net L1: now also J4.1 (L); no longer J4. (PE)
- net L2: now also J4.2 (N); no longer J4. (PE)
Other:
- company: JK&Sons, Engineering -> Scott Dube, In-Tolerance Machine
